Commit message: 完成local-move_base

File: urdf/smart_car.urdf (robot description, URDF)
Before this commit: robot smartcar, 7 links, 6 joints
Links:
- added link gps_link; visual box size=0.001 0.001 0.001
- added link imu_link; visual box size=0.001 0.001 0.001
Joints:
- added joint gps_link_joint: type fixed, parent base_link, child gps_link, origin xyz=0 0 -0.05 rpy=0 0 0
- added joint imu_link_joint: type fixed, parent base_link, child imu_link, origin xyz=0 0 0.05 rpy=0 0 0
